File: schematics/DRAM Board.kicad_pcb (KiCad board)
At the start: 2 copper layers, 114.3 x 53.3 mm, 17 parts, among them U1 AS4C256K16E0, U16 44256_DRAM, U17 44256_DRAM, U18 44256_DRAM, U19 44256_DRAM, U2 AS4C256K16E0, U20 44256_DRAM, U21 44256_DRAM, U22 44256_DRAM, U23 44256_DRAM, U3 AS4C256K16E0, U4 AS4C256K16E0, U5 LM1117-3.3

Commit message: Add files via upload
Routing:
- net /gnd: track 0.00 -> 292.2 mm, vias 0 -> 5
- net /a0: track 0.00 -> 223.4 mm, vias 0 -> 3
- net /a3: track 0.00 -> 222.6 mm, vias 0 -> 2
- net /a2: track 0.00 -> 222.0 mm, vias 0 -> 2
- net /a6: track 0.00 -> 202.9 mm, vias 0 -> 2
- net /a8: track 0.00 -> 200.2 mm, vias 0 -> 3
- net /a7: track 0.00 -> 190.7 mm, vias 0 -> 3
- net /a5: track 0.00 -> 186.9 mm, vias 0 -> 5
- net /_oe: track 0.00 -> 182.9 mm, vias 0 -> 3
- net /_we: track 0.00 -> 182.4 mm, vias 0 -> 4
- net /a4: track 0.00 -> 180.9 mm, vias 0 -> 5
- net /VCC: track 0.00 -> 180.0 mm, vias 0 -> 5
- net /a1: track 0.00 -> 179.1 mm, vias 0 -> 2
- net /vcc5: track 0.00 -> 146.8 mm, vias 0 -> 1
- net /d14: track 0.00 -> 136.6 mm, vias 0 -> 3
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